Commit message: Replace 4-DOF robot with full 7-DOF KUKA IIWA
Copy complete robot structure from pybullet_kuka and update mesh paths.

File: kuka_3dof.urdf (robot description, URDF)
Before this commit: robot lbr_iiwa_3dof, 7 links, 6 joints
Links:
- removed link gripper_body
- added link body, mass 0.988882; collision box size=0.146 0.0725 0.049521; visual box size=0.146 0.0725 0.049521
- added link lbr_iiwa_link_4, mass 2.7; collision mesh filename=pybullet_kuka/kuka_iiwa/meshes/link_4.stl; visual mesh filename=pybullet_kuka/kuka_iiwa/meshes/link_4.obj
- added link lbr_iiwa_link_5, mass 1.7; collision mesh filename=pybullet_kuka/kuka_iiwa/meshes/link_5.stl; visual mesh filename=pybullet_kuka/kuka_iiwa/meshes/link_5.obj
- added link lbr_iiwa_link_6, mass 1.8; collision mesh filename=pybullet_kuka/kuka_iiwa/meshes/link_6.stl; visual mesh filename=pybullet_kuka/kuka_iiwa/meshes/link_6.obj
- added link lbr_iiwa_link_7, mass 0.3; collision mesh filename=pybullet_kuka/kuka_iiwa/meshes/link_7.stl; visual mesh filename=pybullet_kuka/kuka_iiwa/meshes/link_7.obj
Joints:
- removed joint left_finger_joint
- removed joint right_finger_joint
- added joint lbr_iiwa_joint_4: type revolute, parent lbr_iiwa_link_3, child lbr_iiwa_link_4, origin xyz=0 0 0.2155 rpy=1.57079632679 0 0, axis 0 0 1, limit lower=-2.09439510239 upper=2.09439510239 effort=300 velocity=10
- added joint lbr_iiwa_joint_5: type revolute, parent lbr_iiwa_link_4, child lbr_iiwa_link_5, origin xyz=0 0.1845 0 rpy=-1.57079632679 3.14159265359 0, axis 0 0 1, limit lower=-2.96705972839 upper=2.96705972839 effort=300 velocity=10
- added joint lbr_iiwa_joint_6: type revolute, parent lbr_iiwa_link_5, child lbr_iiwa_link_6, origin xyz=0 0 0.2155 rpy=1.57079632679 0 0, axis 0 0 1, limit lower=-2.09439510239 upper=2.09439510239 effort=300 velocity=10
- added joint lbr_iiwa_joint_7: type revolute, parent lbr_iiwa_link_6, child lbr_iiwa_link_7, origin xyz=0 0.081 0 rpy=-1.57079632679 3.14159265359 0, axis 0 0 1, limit lower=-3.05432619099 upper=3.05432619099 effort=300 velocity=10
- added joint left_finger_sliding_joint: type prismatic, parent body, child left_finger, origin xyz=-0.008 0.025 0 rpy=0 0 0, axis 1 0 0, limit lower=-0.055 upper=0 effort=80
- added joint right_finger_sliding_joint: type prismatic, parent body, child right_finger, origin xyz=0.008 0.025 0 rpy=0 0 0, axis 1 0 0, limit lower=0 upper=0.055 effort=80
- joint gripper_base: child gripper_body -> body; origin xyz=0 0 0.2155 rpy=1.57 0 -1.57 -> xyz=0 0 0.13 rpy=1.57 0 -1.57; parent lbr_iiwa_link_3 -> lbr_iiwa_link_7
- joint lbr_iiwa_joint_2: origin xyz=0 0 0.2025 rpy=1.57079632679 0 3.14159265359 -> xyz=0 0 0.2025 rpy=1.57079632679   0 3.14159265359
